Commit message: modify wheel

File: simple_yolo_tracker_Version2.urdf (robot description, URDF)
Before this commit: robot simple_yolo_tracker, 4 links, 3 joints
Joints:
- joint camera_joint: origin xyz=0.15 0 0.06 rpy=0 0 0 -> xyz=0.15 0 0.09 rpy=0 0 0
- joint left_wheel_joint: origin xyz=0.12 0.09 0 rpy=0 0 0 -> xyz=0.0 0.11 0.05 rpy=0 0 0
- joint right_wheel_joint: origin xyz=0.12 -0.09 0 rpy=0 0 0 -> xyz=0.0 -0.11 0.05 rpy=0 0 0
