Commit message: modify wheel

File: simple_yolo_tracker_Version4.urdf (robot description, URDF)
Before this commit: robot simple_yolo_tracker, 4 links, 3 joints
Joints:
- joint left_wheel_joint: origin xyz=0.0 0.12 0.05 rpy=0 0 0 -> xyz=0 0.12 0.05 rpy=0 0 0
- joint right_wheel_joint: origin xyz=0.0 -0.12 0.05 rpy=0 0 0 -> xyz=0 -0.12 0.05 rpy=0 0 0

Commit message: modify wheel

File: simple_yolo_tracker_Version4.urdf (robot description, URDF)
Before this commit: robot simple_yolo_tracker, 4 links, 3 joints
Joints:
- joint camera_joint: origin xyz=0.15 0 0.09 rpy=0 0 0 -> xyz=0 0.15 0.09 rpy=0 0 0
- joint left_wheel_joint: axis 0 1 0 -> 1 0 0; origin xyz=0 0.12 0.05 rpy=0 0 0 -> xyz=0.12 0 0.05 rpy=0 0 0
- joint right_wheel_joint: axis 0 1 0 -> 1 0 0; origin xyz=0 -0.12 0.05 rpy=0 0 0 -> xyz=-0.12 0 0.05 rpy=0 0 0

Commit message: modify wheel

File: simple_yolo_tracker_Version4.urdf (robot description, URDF)
Before this commit: robot simple_yolo_tracker, 4 links, 3 joints
Joints:
- joint camera_joint: origin xyz=0 0.15 0.09 rpy=0 0 0 -> xyz=0.15 0 0.09 rpy=0 0 0
- joint left_wheel_joint: axis 1 0 0 -> 0 1 0; origin xyz=0.12 0 0.05 rpy=0 0 0 -> xyz=0 0.12 0.05 rpy=0 0 0
- joint right_wheel_joint: axis 1 0 0 -> 0 1 0; origin xyz=-0.12 0 0.05 rpy=0 0 0 -> xyz=0 -0.12 0.05 rpy=0 0 0

Commit message: modify wheel

File: simple_yolo_tracker_Version4.urdf (robot description, URDF)
Before this commit: robot simple_yolo_tracker, 5 links, 4 joints
Links:
- link base_link: geometry collision box size=0.3 0.2 0.06; visual box size=0.3 0.2 0.06
Joints:
- joint camera_joint: origin xyz=0.15 0 0.09 rpy=0 0 0 -> xyz=0.15 0 0.13 rpy=0 0 0
